File: kicad/baseboard/baseboard.kicad_sch (KiCad schematic)
At the start: 4 parts, among them J2 10164227-1001A1RLF, J6 10164227-1001A1RLF

Commit message: Finish PCB routing
Parts:
- added H1, H2, H3, H4: MountingHole, MountingHole:MountingHole_3.2mm_M3_DIN965, symbol Mechanical:MountingHole
- C18, C9: footprint Capacitor_SMD:C_0402_1005Metric -> Capacitor_SMD:C_0603_1608Metric; LCSC Part # (none) -> C14663
- J2, J6: LCSC Part # (none) -> C7435219; j C6782225 -> (none)
